File: Diplom/Diplom.kicad_pcb (KiCad board)
At the start: 2 copper layers, 100 x 80 mm, 94 parts, among them IC1 E22-900T22D, J1 Conn_01x03_Pin, J2 Conn_01x05_Pin, J3 Conn_01x02_Pin, Q1 SI2301, SW1 SW_Push, SW2 SW_Push, U2 BME280, U3 W25Q32JVSS, U4 SPV1040, U5 DW01A, U6 STM32F411CEUx, Y3 ABM3-25.000MHz-D2Y-T, Y4 KX-327NHT, Y5 Crystal

Commit message: Corr
Parts:
- moved C23 2.74 mm to (94.0, 58.9)
- moved C24 2.74 mm to (92.5, 58.9)
- moved C25 2.74 mm to (91.0, 58.9)
Routing:
- net /MCU/AXEL_SCK: track 31.2 -> 30.6 mm
Changed lines of the file:
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@@
 		(tenting front back)
 		(pcbplotparams
-			(layerselection 0x00000000_00000000_55555555_5755f5f5)
-			(plot_on_all_layers_selection 0x00000000_00000000_00000000_02000000)
+			(layerselection 0x00000000_00000000_55555555_5755f5ff)
+			(plot_on_all_layers_selection 0x00000000_00000000_00000000_00000000)
 			(disableapertmacros no)
 			(usegerberextensions no)
@@
 		(tags "resistor handsolder")
 		(property "Reference" "R18"
-			(at 4.4 -0.33 0)
+			(at -0.030001 -1.879999 0)
 			(layer "F.SilkS")
 			(effects
@@
 		(tags "capacitor handsolder")
 		(property "Reference" "C36"
-			(at 3.5 0 90)
+			(at -4.25 0 90)
 			(layer "F.SilkS")
 			(effects
@@
 	(footprint "Capacitor_SMD:C_0603_1608Metric_Pad1.08x0.95mm_HandSolder"
 		(layer "F.Cu")
-		(at 89.4 61.1 90)
+		(at 90.976 58.862501 90)
 		(descr "Capacitor SMD 0603 (1608 Metric), square (rectangular) end terminal, IPC-7351 nominal with elongated pad for handsoldering. (Body size source: IPC-SM-782 page 76, https://www.pcb-3d.com/wordpress/wp-content/uploads/ipc-sm-782a_amendment_1_and_2.pdf), generated with kicad-footprint-generator")
 		(tags "capacitor handsolder")
 		(property "Reference" "C25"
-			(at -3.32 -0.076 90)
+			(at 3.362501 0 90)
 			(layer "F.SilkS")
 			(effects
@@
 	(footprint "Capacitor_SMD:C_0603_1608Metric_Pad1.08x0.95mm_HandSolder"
 		(layer "F.Cu")
-		(at 90.924 61.1 90)
+		(at 92.5 58.862501 90)
 		(descr "Capacitor SMD 0603 (1608 Metric), square (rectangular) end terminal, IPC-7351 nominal with elongated pad for handsoldering. (Body size source: IPC-SM-782 page 76, https://www.pcb-3d.com/wordpress/wp-content/uploads/ipc-sm-782a_amendment_1_and_2.pdf), generated with kicad-footprint-generator")
 		(tags "capacitor handsolder")
 		(property "Reference" "C24"
-			(at -3.23 0.02 90)
+			(at 3.362501 0 90)
 			(layer "F.SilkS")
 			(effects
@@
 	(footprint "Capacitor_SMD:C_0603_1608Metric_Pad1.08x0.95mm_HandSolder"
 		(layer "F.Cu")
-		(at 92.448 61.1 90)
+		(at 94.024 58.862501 90)
 		(descr "Capacitor SMD 0603 (1608 Metric), square (rectangular) end terminal, IPC-7351 nominal with elongated pad for handsoldering. (Body size source: IPC-SM-782 page 76, https://www.pcb-3d.com/wordpress/wp-content/uploads/ipc-sm-782a_amendment_1_and_2.pdf), generated with kicad-footprint-generator")
 		(tags "capacitor handsolder")
 		(property "Reference" "C23"
-			(at -3.23 0.096 90)
+			(at 3.362501 -0.024 90)
 			(layer "F.SilkS")
 			(effects
@@
 	)
 	(segment
-		(start 90.924 60.237499)
-		(end 90.924 58.48)
+		(start 92.5 58)
+		(end 92.5 56.242501)
 		(width 0.508)
 		(layer "F.Cu")
@@
 	)
 	(segment
-		(start 89.4 60.237499)
-		(end 92.448 60.237499)
+		(start 90.976 58)
+		(end 94.024 58)
 		(width 0.508)
 		(layer "F.Cu")
@@
 	)
 	(via
-		(at 90.924 58.48)
+		(at 92.5 56.242501)
 		(size 0.7)
 		(drill 0.3)
@@
 	)
 	(segment
-		(start 108 70.75)
-		(end 107.5 71.25)
-		(width 0.2)
-		(layer "F.Cu")
-		(net 58)
-	)
-	(segment
-		(start 110.25 70.5)
-		(end 110 70.75)
+		(start 97 67.25)
+		(end 97.5 67.75)
 		(width 0.2)
 		(layer "F.Cu")
@@
 	)
 	(segment
-		(start 110 70.75)
-		(end 108 70.75)
+		(start 112.45 80.05)
+		(end 114 78.5)
 		(width 0.2)
 		(layer "F.Cu")
@@
 	)
 	(segment
-		(start 97 67.25)
-		(end 97.5 67.75)
+		(start 111.5 71.5)
+		(end 111.25 71.25)
 		(width 0.2)
 		(layer "F.Cu")
@@
 	)
 	(segment
-		(start 112.45 80.05)
-		(end 114 78.5)
+		(start 111.25 71.25)
+		(end 107.5 71.25)
 		(width 0.2)
 		(layer "F.Cu")
@@
 	)
 	(via
-		(at 110.25 70.5)
+		(at 111.5 71.5)
 		(size 0.6)
 		(drill 0.3)
@@
 	)
 	(segment
-		(start 107.5 71.25)
-		(end 101 71.25)
-		(width 0.2)
-		(layer "B.Cu")
-		(net 58)
-	)
-	(segment
-		(start 114 78.5)
-		(end 114.25 78.25)
+		(start 114.25 78.25)
+		(end 114 78.5)
 		(width 0.2)
 		(layer "B.Cu")
@@
 	)
 	(segment
-		(start 110.5 70.5)
-		(end 110.25 70.5)
+		(start 107.5 71.25)
+		(end 101 71.25)
 		(width 0.2)
 		(layer "B.Cu")
@@
 	(segment
 		(start 114.25 74.25)
-		(end 110.5 70.5)
+		(end 114.25 78.25)
 		(width 0.2)
 		(layer "B.Cu")
@@
 	)
 	(segment
-		(start 114.25 78.25)
+		(start 111.5 71.5)
 		(end 114.25 74.25)
 		(width 0.2)
